File: sensors/pcb/airball_sensors/airball_sensors.sch (KiCad schematic (older format))
At the start: 14 parts, among them U1 PWM3360_Motion_Sensor, U2 PWM3360_Motion_Sensor

Commit message: PCB v1.1
Connections:
- net +5V: now also XA2.5V, XA3.5V
- net GND: now also XA1.GND2 (GND), XA1.GND3 (GND), XA1.GND5 (GND), XA1.GND6 (GND), XA2.GND2 (GND), XA3.GND2 (GND)
- no-connect marks 136 -> 128
Changed lines of the file:
@@
 NoConn ~ 1600 5550
 NoConn ~ 1600 5350
-NoConn ~ 1600 5250
-NoConn ~ 1600 5150
-NoConn ~ 1600 5050
-NoConn ~ 1600 4950
 NoConn ~ 1600 4650
 NoConn ~ 1600 4550
@@
 NoConn ~ 8900 3000
 NoConn ~ 6300 2900
-NoConn ~ 6300 2800
 NoConn ~ 6300 2500
 NoConn ~ 6300 2400
@@
 NoConn ~ 6300 1600
 NoConn ~ 6300 1300
-NoConn ~ 6300 5450
 NoConn ~ 6300 5550
 $Comp
@@
 	0    -1   -1   0
 $EndComp
-NoConn ~ 6300 3000
-NoConn ~ 6300 5650
 $Comp
 L R 1k4
@@
 	8900 2400 9150 2400
 Connection ~ 9050 2400
+$Comp
+L GND #PWR024
+U 1 1 5F60DB6F
+P 1600 4950
+F 0 "#PWR024" H 1600 4700 50  0001 C CNN
+F 1 "GND" H 1600 4800 50  0000 C CNN
+F 2 "" H 1600 4950 50  0001 C CNN
+F 3 "" H 1600 4950 50  0001 C CNN
+	1    1600 4950
+	0    1    1    0
+$EndComp
+$Comp
+L GND #PWR025
+U 1 1 5F60DB9F
+P 1600 5050
+F 0 "#PWR025" H 1600 4800 50  0001 C CNN
+F 1 "GND" H 1600 4900 50  0000 C CNN
+F 2 "" H 1600 5050 50  0001 C CNN
+F 3 "" H 1600 5050 50  0001 C CNN
+	1    1600 5050
+	0    1    1    0
+$EndComp
+$Comp
+L GND #PWR026
+U 1 1 5F60DBCF
+P 1600 5150
+F 0 "#PWR026" H 1600 4900 50  0001 C CNN
+F 1 "GND" H 1600 5000 50  0000 C CNN
+F 2 "" H 1600 5150 50  0001 C CNN
+F 3 "" H 1600 5150 50  0001 C CNN
+	1    1600 5150
+	0    1    1    0
+$EndComp
+$Comp
+L GND #PWR027
+U 1 1 5F60DBFF
+P 1600 5250
+F 0 "#PWR027" H 1600 5000 50  0001 C CNN
+F 1 "GND" H 1600 5100 50  0000 C CNN
+F 2 "" H 1600 5250 50  0001 C CNN
+F 3 "" H 1600 5250 50  0001 C CNN
+	1    1600 5250
+	0    1    1    0
+$EndComp
+$Comp
+L GND #PWR028
+U 1 1 5F60DE99
+P 6300 2800
+F 0 "#PWR028" H 6300 2550 50  0001 C CNN
+F 1 "GND" H 6300 2650 50  0000 C CNN
+F 2 "" H 6300 2800 50  0001 C CNN
+F 3 "" H 6300 2800 50  0001 C CNN
+	1    6300 2800
+	0    1    1    0
+$EndComp
+$Comp
+L GND #PWR029
+U 1 1 5F60DED9
+P 6300 5450
+F 0 "#PWR029" H 6300 5200 50  0001 C CNN
+F 1 "GND" H 6300 5300 50  0000 C CNN
+F 2 "" H 6300 5450 50  0001 C CNN
+F 3 "" H 6300 5450 50  0001 C CNN
+	1    6300 5450
+	0    1    1    0
+$EndComp
+$Comp
+L +5V #PWR030
+U 1 1 5F60E1F1
+P 6300 5650
+F 0 "#PWR030" H 6300 5500 50  0001 C CNN
+F 1 "+5V" H 6300 5790 50  0000 C CNN
+F 2 "" H 6300 5650 50  0001 C CNN
+F 3 "" H 6300 5650 50  0001 C CNN
+	1    6300 5650
+	0    -1   -1   0
+$EndComp
+$Comp
+L +5V #PWR031
+U 1 1 5F60E231
+P 6300 3000
+F 0 "#PWR031" H 6300 2850 50  0001 C CNN
+F 1 "+5V" H 6300 3140 50  0000 C CNN
+F 2 "" H 6300 3000 50  0001 C CNN
+F 3 "" H 6300 3000 50  0001 C CNN
+	1    6300 3000
+	0    -1   -1   0
+$EndComp
 $EndSCHEMATC
