File: sensors/pcb/file_for_printing/airball_sensors.kicad_pcb (KiCad board)
At the start: 2 copper layers, 144.8 x 59.7 mm, 15 parts, among them U1 PWM3360_Motion_Sensor, U2 PWM3360_Motion_Sensor

Commit message: PCB v1.1
Parts:
- removed .1u (x2), 10u: C, Capacitors_THT:C_Disc_D6.0mm_W2.5mm_P5.00mm
- removed 1k (x4), 2k (x2): R, Resistors_THT:R_Axial_DIN0207_L6.3mm_D2.5mm_P7.62mm_Horizontal
- removed G***: LOGO, footprints:nerf_logo
- added 0.1uF1: C, Capacitors_THT:C_Disc_D6.0mm_W2.5mm_P5.00mm, F.Cu at (111.1, 96.5)
- added 0.1uF2: C, Capacitors_THT:C_Disc_D6.0mm_W2.5mm_P5.00mm, F.Cu at (132.1, 96.5)
- added 10uF1: C, Capacitors_THT:C_Disc_D6.0mm_W2.5mm_P5.00mm, F.Cu at (194.9, 91.4)
- added 1k1: R, Resistors_THT:R_Axial_DIN0207_L6.3mm_D2.5mm_P7.62mm_Horizontal, F.Cu at (159.4, 128.3)
- added 1k2: R, Resistors_THT:R_Axial_DIN0207_L6.3mm_D2.5mm_P7.62mm_Horizontal, F.Cu at (164.5, 128.3)
- added 1k3: R, Resistors_THT:R_Axial_DIN0207_L6.3mm_D2.5mm_P7.62mm_Horizontal, F.Cu at (116.8, 82.5)
- added 1k4: R, Resistors_THT:R_Axial_DIN0207_L6.3mm_D2.5mm_P7.62mm_Horizontal, F.Cu at (184.8, 83.2)
- added 2k1: R, Resistors_THT:R_Axial_DIN0207_L6.3mm_D2.5mm_P7.62mm_Horizontal, F.Cu at (151.8, 131.4)
- added 2k2: R, Resistors_THT:R_Axial_DIN0207_L6.3mm_D2.5mm_P7.62mm_Horizontal, F.Cu at (164.5, 131.4)
Connections:
- XA1 pad GND2: (no net) -> GND
- XA1 pad GND3: (no net) -> GND
- XA1 pad GND5: (no net) -> GND
- XA1 pad GND6: (no net) -> GND
- XA2 pad 5V: (no net) -> +5V
- XA2 pad GND2: (no net) -> GND
- XA3 pad 5V: (no net) -> +5V
- XA3 pad GND2: (no net) -> GND
Routing:
- net +5V: track 79.0 -> 181.3 mm
- net /TX_MICRO_2: track 123.5 -> 117.8 mm, vias 2 -> 4
- net +12V: track 117.5 -> 113.2 mm
- net /MT_2: track 71.3 -> 72.3 mm
- net /SS_2: track 68.4 -> 69.3 mm
- net /SS_1: track 69.6 -> 70.0 mm, vias 2 -> 4
- net /MT_1: track 68.2 -> 68.6 mm, vias 2 -> 4
Other:
- outline, holes or cut-outs redrawn
- board text added: "Adrien Philippon 2020"
- board text added: "AirBall PCB v1.1"
- board text removed: "Adrien Philippon 2019"
- board text removed: "AirBall PCB v1.0"
